File: Garden-MUX/Garden-MUX.kicad_sch (KiCad schematic)
At the start: 80 parts, among them J3 SDCARD_MODULE, J4 USB_C_Receptacle_USB2.0_16P, P1 S2B-PH-SM4-TB, Q1 AO3401A, U1 MCP73832-2-OT, U2 ESP32-S2, U3 AP2112K-3.3, U4 AP2112K-3.3, Y1 40MHz

Commit message: initial changes
Parts:
- renumbered C16 to C10, C19 to C11, C17 to C12, C27 to C13, C21 to C14, C28 to C15, C22 to C16, C23 to C17, C24 to C18, C10 to C19, C9 to C20, C11 to C21, C31 to C22, C12 to C23, C13 to C24, C29 to C25, C14 to C26, C30 to C27, C20 to C5, C15 to C6, C25 to C7, C26 to C8, C18 to C9, D3 to D2, D2 to D3, J4 to J1, J3 to J2, L2 to L1, L1 to L2, R26 to R1, R22 to R10, R23 to R11, R30 to R12, R31 to R13, R32 to R14, R35 to R15, R24 to R16, R25 to R17, R34 to R18, R33 to R19, R19 to R2, R17 to R3, R18 to R4, R27 to R5, R20 to R6, R28 to R7, R21 to R8, R29 to R9, S9 to S10, S10 to S9, U2 to U1, U1 to U2

Commit message: Add missing May changes
Parts:
- removed C10, C11, C12: 0.1, Capacitor_SMD:C_0603_1608Metric, symbol Device:C_Small
- removed C13, C15: TBA, Capacitor_SMD:C_0805_2012Metric, symbol Device:C
- removed C14, C6: 0.1, Capacitor_SMD:C_0603_1608Metric, symbol Device:C
- removed C16: 22, Capacitor_SMD:C_0805_2012Metric, symbol Device:C
- removed C17, C18, C27: 1, Capacitor_SMD:C_0603_1608Metric, symbol Device:C
- removed C22: 10, Capacitor_SMD:C_0603_1608Metric, symbol Device:C
- removed C7, C8: 16, Capacitor_SMD:C_0805_2012Metric, symbol Device:C_Small
- removed C9: 1, Capacitor_SMD:C_0603_1608Metric, symbol Device:C_Small
- removed E1: ANTENNA, Pico_Footprints:ANTENNA_Footprint, symbol Pico_Symbols:ANTENNA
- removed JP1, JP2, JP3: SolderJumper_2_Open, Jumper:SolderJumper-2_P1.3mm_Open_TrianglePad1.0x1.5mm, symbol Jumper:SolderJumper_2_Open
- removed L1: TBA, Inductor_SMD:L_APV_ANR3015, symbol Device:L
- removed L2: 2nH, Inductor_SMD:L_0603_1608Metric, symbol Device:L
- removed R1, R5, R7, R9: 10k, Resistor_SMD:R_0603_1608Metric, symbol Device:R_US
- removed S10: ~, Pico_Footprints:STEMMAQWIIC_Footprint, symbol Pico_Symbols:STEMMA_QT
- removed S9: TL6330AF200Q, Pico_Footprints:SW_TL6330AF200Q_Footprint, symbol Pico_Symbols:TL6330AF200Q
- removed TP1: RESET PIN, TestPoint:TestPoint_THTPad_1.0x1.0mm_Drill0.5mm, symbol Connector:TestPoint
- removed U1: ESP32-S2, Package_DFN_QFN:QFN-56-1EP_7x7mm_P0.4mm_EP4x4mm_ThermalVias, symbol MCU_Espressif:ESP32-S2
- removed Y1: 40MHz, Crystal:Crystal_SMD_2016-4Pin_2.0x1.6mm, symbol Device:Crystal_GND24
- added R20: 5.1k, Resistor_SMD:R_0603_1608Metric, symbol Device:R_US
- added S11: TL6330AF200Q, Pico_Footprints:SW_TL6330AF200Q_Footprint, symbol Pico_Symbols:TL6330AF200Q
- added U5: ESP32-C6-MINI-1, RF_Module:ESP32-C6-MINI-1, symbol RF_Module:ESP32-C6-MINI-1
- C25: value 1 -> 10
Connections:
- net A0 is gone; now on net GND: TCA9548A1.21 (A2)
- net A1 is gone; now on net GND: TCA9548A1.2 (A1)
- net A2 is gone; now on net GND: TCA9548A1.1 (A0)
- net RESET is gone; now on net GND: TCA9548A1.3 (#RESET)
- net VDD_SPI is gone; now on net RST: C5.1
- net +3.3V: now also R20.1, U5.3 (3V3); no longer C19.1, C20.1, C26.1, J2.4 (VDD), R10.1, R11.1, R16.1, R17.1, R2.1, R4.1, R6.1, R8.1
- net +BATT: now also C26.1
- net 3.3V_I2C: now also C19.1, C20.1, J2.4 (VDD), R10.1, R11.1, R16.1, R17.1, R2.1, R4.1, R6.1, R8.1
- net CS: now also U5.25 (IO19)
- net DAT1: now also U5.29 (IO23)
- net DAT2: now also U5.24 (IO18)
- net DATA_IN: now also U5.26 (IO20)
- net DATA_OUT: now also U5.28 (IO22)
- net GND: now also S11.1, S11.2, U5.1 (GND), U5.11 (GND), U5.14 (GND), U5.2 (GND), U5.36 (GND), U5.37 (GND), U5.38 (GND), U5.39 (GND), U5.40 (GND), U5.41 (GND), U5.42 (GND), U5.43 (GND), U5.44 (GND), U5.45 (GND), U5.46 (GND), U5.47 (GND), U5.48 (GND), U5.49 (GND), U5.50 (GND), U5.51 (GND), U5.52 (GND), U5.53 (GND)
- net I2C_POWER: now also U5.19 (IO14)
- net MUX_SCL: now also U5.16 (IO7)
- net MUX_SDA: now also U5.15 (IO6)
- net RST: now also R20.2, S11.3, S11.4, U5.8 (EN)
- net SD_CLK: now also U5.27 (IO21)
- net USB_D+: now also U5.18 (IO13)
- net USB_D-: now also U5.17 (IO12)
- no-connect marks 9 -> 3
Other:
- note added: "ESP32 C6 CONNECTIONS"
- note removed: "ESP32 S2 CONNECTIONS"
- moved on the sheet: H1, H2, H3, H4
